File: master_schematic/master_schematic.kicad_pcb (KiCad board)
At the start: 4 copper layers, 157.5 x 111.9 mm, 69 parts, among them J1 Conn_01x02_Shielded, J10 0430450400, J11 1723103102, J12 1723103102, J13 1723103102, J14 1723103102, J15 1723103102, J16 1723103102, J17 1723103102, J18 1723103102, J19 1723103102, J2 0430450400, J3 0430450400, J4 0430450400, J5 0430450400, J6 0430450400, J7 0430450400, J8 0430450400, J9 0430450400, Q1 CWDM3011N TR13 PBFREE, Q2 CWDM3011N TR13 PBFREE, Q3 CWDM3011N TR13 PBFREE, Q4 CWDM3011N TR13 PBFREE, Q5 CWDM3011N TR13 PBFREE, Q6 CWDM3011N TR13 PBFREE, Q7 CWDM3011N TR13 PBFREE, Q8 CWDM3011N TR13 PBFREE, Q9 CWDM3011N TR13 PBFREE, U1 teensy_4.1, U10 HX711, U11 HX711, U2 RFM95, U4 MCP9600_Module, U5 MCP9600_Module, U6 MCP9600_Module, U7 MCP9600_Module, U8 MCP9600_Module, U9 HX711

Commit message: updated BOM
Parts:
- added U10: HX711, hb_footprint_lib:hx711_connector, F.Cu at (39.9, 0.25)
- added U11: HX711, hb_footprint_lib:hx711_connector, F.Cu at (39.9, 24.4)
- added U5: MCP9600_Module, hb_footprint_lib:mcp9600_connector, F.Cu at (12.7, 0.25)
- added U6: MCP9600_Module, hb_footprint_lib:mcp9600_connector, F.Cu at (12.7, 21.8)
- added U7: MCP9600_Module, hb_footprint_lib:mcp9600_connector, F.Cu at (12.7, 43.4)
- added U8: MCP9600_Module, hb_footprint_lib:mcp9600_connector, F.Cu at (12.7, 65.0)
