File: master_schematic/master_schematic.kicad_pcb (KiCad board)
At the start: 4 copper layers, 81.5 x 88 mm, 4 parts, among them U1 teensy_4.1

Commit message: fixed errors on schematic
Parts:
- removed PT1: ~, hb_footprint_lib:Pressure Transducer (Low)
- removed RM1: ~, hb_footprint_lib:Radio_Module
- removed U1: teensy_4.1, hb_footprint_lib:teensy4.1
- removed U4: ~, Connector_PinHeader_1.00mm:PinHeader_1x06_P1.00mm_Vertical
Routing:
- net /5V: track 5.21 -> 0.00 mm, vias 1 -> 0
- net /GND: track 1.99 -> 0.00 mm, vias 1 -> 0
- removed copper zone on In1.Cu, net /GND
Other:
- board outline removed

Commit message: finished building PCB
Parts:
- added D1: SBRT20U60SP5-7, hb_footprint_lib:POWERDI5_DIO, F.Cu at (143.0, 47.5)
- added D2: SBRT20U60SP5-7, hb_footprint_lib:POWERDI5_DIO, F.Cu at (135.5, 47.4)
- added D3: SBRT20U60SP5-7, hb_footprint_lib:POWERDI5_DIO, F.Cu at (127.2, 47.4)
- added D4: SBRT20U60SP5-7, hb_footprint_lib:POWERDI5_DIO, F.Cu at (118.8, 47.4)
- added D5: SBRT20U60SP5-7, hb_footprint_lib:POWERDI5_DIO, F.Cu at (110.4, 47.4)
- added D6: SBRT20U60SP5-7, hb_footprint_lib:POWERDI5_DIO, F.Cu at (102.0, 47.5)
- added D7: SBRT20U60SP5-7, hb_footprint_lib:POWERDI5_DIO, F.Cu at (93.6, 47.5)
- added D8: SBRT20U60SP5-7, hb_footprint_lib:POWERDI5_DIO, F.Cu at (85.2, 47.4)
- added D9: SBRT20U60SP5-7, hb_footprint_lib:POWERDI5_DIO, F.Cu at (76.8, 47.4)
- added H1: MountingHole, MountingHole:MountingHole_4.3mm_M4_DIN965_Pad, F.Cu at (32.0, 28.0)
- added H2: MountingHole, MountingHole:MountingHole_4.3mm_M4_DIN965_Pad, F.Cu at (175.5, 28.0)
- added H3: MountingHole, MountingHole:MountingHole_4.3mm_M4_DIN965_Pad, F.Cu at (32.0, 125.9)
- added H4: MountingHole, MountingHole:MountingHole_4.3mm_M4_DIN965_Pad, F.Cu at (175.5, 125.9)
- added J1: Conn_01x02_Shielded, hb_footprint_lib:AMASS_XT60PW-M, F.Cu at (172.0, 53.2)
- added J10: 0430450400, hb_footprint_lib:CONN_SD-43045-001_04_MOL, F.Cu at (161.5, 123.8)
- added J11: 1723103102, hb_footprint_lib:CONN02_1723103102_MOL, F.Cu at (163.4, 36.4)
- added J12: 1723103102, hb_footprint_lib:CONN02_1723103102_MOL, F.Cu at (149.0, 36.4)
- added J13: 1723103102, hb_footprint_lib:CONN02_1723103102_MOL, F.Cu at (134.5, 36.4)
- added J14: 1723103102, hb_footprint_lib:CONN02_1723103102_MOL, F.Cu at (120.1, 36.4)
- added J15: 1723103102, hb_footprint_lib:CONN02_1723103102_MOL, F.Cu at (105.6, 36.4)
- added J16: 1723103102, hb_footprint_lib:CONN02_1723103102_MOL, F.Cu at (91.2, 36.4)
- added J17: 1723103102, hb_footprint_lib:CONN02_1723103102_MOL, F.Cu at (76.7, 36.4)
- added J18: 1723103102, hb_footprint_lib:CONN02_1723103102_MOL, F.Cu at (62.3, 36.4)
- added J19: 1723103102, hb_footprint_lib:CONN02_1723103102_MOL, F.Cu at (47.9, 36.4)
- added J2: 0430450400, hb_footprint_lib:CONN_SD-43045-001_04_MOL, F.Cu at (49.1, 123.8)
- added J3: 0430450400, hb_footprint_lib:CONN_SD-43045-001_04_MOL, F.Cu at (63.1, 123.8)
- added J4: 0430450400, hb_footprint_lib:CONN_SD-43045-001_04_MOL, F.Cu at (77.2, 123.8)
- added J5: 0430450400, hb_footprint_lib:CONN_SD-43045-001_04_MOL, F.Cu at (91.2, 123.8)
- added J6: 0430450400, hb_footprint_lib:CONN_SD-43045-001_04_MOL, F.Cu at (105.3, 123.8)
- added J7: 0430450400, hb_footprint_lib:CONN_SD-43045-001_04_MOL, F.Cu at (119.3, 123.8)
- added J8: 0430450400, hb_footprint_lib:CONN_SD-43045-001_04_MOL, F.Cu at (133.4, 123.8)
- added J9: 0430450400, hb_footprint_lib:CONN_SD-43045-001_04_MOL, F.Cu at (147.4, 123.8)
- added Q1: CWDM3011N TR13 PBFREE, Package_SO:SOIC-8_3.9x4.9mm_P1.27mm, F.Cu at (143.7, 58.4)
- added Q2: CWDM3011N TR13 PBFREE, Package_SO:SOIC-8_3.9x4.9mm_P1.27mm, F.Cu at (135.0, 58.4)
- added Q3: CWDM3011N TR13 PBFREE, Package_SO:SOIC-8_3.9x4.9mm_P1.27mm, F.Cu at (126.4, 58.4)
- added Q4: CWDM3011N TR13 PBFREE, Package_SO:SOIC-8_3.9x4.9mm_P1.27mm, F.Cu at (117.8, 58.4)
- added Q5: CWDM3011N TR13 PBFREE, Package_SO:SOIC-8_3.9x4.9mm_P1.27mm, F.Cu at (109.2, 58.4)
- added Q6: CWDM3011N TR13 PBFREE, Package_SO:SOIC-8_3.9x4.9mm_P1.27mm, F.Cu at (100.5, 58.4)
- added Q7: CWDM3011N TR13 PBFREE, Package_SO:SOIC-8_3.9x4.9mm_P1.27mm, F.Cu at (91.9, 58.4)
- added Q8: CWDM3011N TR13 PBFREE, Package_SO:SOIC-8_3.9x4.9mm_P1.27mm, F.Cu at (83.3, 58.4)
- added Q9: CWDM3011N TR13 PBFREE, Package_SO:SOIC-8_3.9x4.9mm_P1.27mm, F.Cu at (74.7, 58.4)
- added R1: 1K, Resistor_SMD:R_0805_2012Metric_Pad1.20x1.40mm_HandSolder, F.Cu at (50.0, 116.9)
- added R10: 2.7K, Resistor_SMD:R_0805_2012Metric_Pad1.20x1.40mm_HandSolder, F.Cu at (102.0, 117.0)
- added R11: 1K, Resistor_SMD:R_0805_2012Metric_Pad1.20x1.40mm_HandSolder, F.Cu at (120.0, 116.9)
- added R12: 2.7K, Resistor_SMD:R_0805_2012Metric_Pad1.20x1.40mm_HandSolder, F.Cu at (116.0, 116.9)
- added R13: 1K, Resistor_SMD:R_0805_2012Metric_Pad1.20x1.40mm_HandSolder, F.Cu at (134.0, 116.9)
- added R14: 2.7K, Resistor_SMD:R_0805_2012Metric_Pad1.20x1.40mm_HandSolder, F.Cu at (130.0, 116.9)
- added R15: 1K, Resistor_SMD:R_0805_2012Metric_Pad1.20x1.40mm_HandSolder, F.Cu at (148.0, 116.9)
- added R16: 2.7K, Resistor_SMD:R_0805_2012Metric_Pad1.20x1.40mm_HandSolder, F.Cu at (144.0, 116.9)
- added R17: 1K, Resistor_SMD:R_0805_2012Metric_Pad1.20x1.40mm_HandSolder, F.Cu at (162.2, 116.9)
- added R18: 2.7K, Resistor_SMD:R_0805_2012Metric_Pad1.20x1.40mm_HandSolder, F.Cu at (158.0, 116.9)
- added R2: 2.7K, Resistor_SMD:R_0805_2012Metric_Pad1.20x1.40mm_HandSolder, F.Cu at (46.0, 116.9)
- added R3: 1K, Resistor_SMD:R_0805_2012Metric_Pad1.20x1.40mm_HandSolder, F.Cu at (64.0, 116.9)
- added R4: 2.7K, Resistor_SMD:R_0805_2012Metric_Pad1.20x1.40mm_HandSolder, F.Cu at (60.0, 116.9)
- added R5: 1K, Resistor_SMD:R_0805_2012Metric_Pad1.20x1.40mm_HandSolder, F.Cu at (78.0, 116.9)
- added R6: 2.7K, Resistor_SMD:R_0805_2012Metric_Pad1.20x1.40mm_HandSolder, F.Cu at (74.0, 116.9)
- added R7: 1K, Resistor_SMD:R_0805_2012Metric_Pad1.20x1.40mm_HandSolder, F.Cu at (92.0, 116.9)
- added R8: 2.7K, Resistor_SMD:R_0805_2012Metric_Pad1.20x1.40mm_HandSolder, F.Cu at (88.0, 116.9)
- added R9: 1K, Resistor_SMD:R_0805_2012Metric_Pad1.20x1.40mm_HandSolder, F.Cu at (106.0, 116.9)
- added U1: teensy_4.1, hb_footprint_lib:teensy4.1, F.Cu at (60.0, 79.1)
- added U10: HX711, hb_footprint_lib:hx711_connector, F.Cu at (168.0, 66.2)
- added U11: HX711, hb_footprint_lib:hx711_connector, F.Cu at (106.2, 66.3)
- added U2: RFM95, hb_footprint_lib:rfm95_connector, F.Cu at (24.0, 57.5)
- added U4: MCP9600_Module, hb_footprint_lib:mcp9600_connector, F.Cu at (47.8, 92.7)
- added U5: MCP9600_Module, hb_footprint_lib:mcp9600_connector, F.Cu at (75.6, 92.7)
- added U6: MCP9600_Module, hb_footprint_lib:mcp9600_connector, F.Cu at (103.3, 92.7)
- added U7: MCP9600_Module, hb_footprint_lib:mcp9600_connector, F.Cu at (131.1, 92.7)
- added U8: MCP9600_Module, hb_footprint_lib:mcp9600_connector, F.Cu at (158.8, 92.7)
- added U9: HX711, hb_footprint_lib:hx711_connector, F.Cu at (136.5, 66.2)
Other:
- board outline added: 157.5 x 111.9 mm

Commit message: pcb layout and traces made (partially)
Parts:
- moved D9 16.0 mm to (60.8, 47.4)
- moved D1 12.9 mm to (155.9, 47.5)
- moved Q9 12.7 mm to (62.0, 58.4)
- moved D8 12.5 mm to (72.7, 47.4)
- moved Q1 12.2 mm to (155.8, 58.4)
- moved Q8 9.57 mm to (73.7, 58.4)
- moved Q2 9.07 mm to (144.1, 58.4)
- moved D7 9.02 mm to (84.6, 47.5)
- moved D2 8.47 mm to (144.0, 47.4)
- moved Q7 6.46 mm to (85.4, 58.4)
- moved Q3 5.96 mm to (132.4, 58.4)
- moved D6 5.52 mm to (96.5, 47.5)
- moved D3 4.97 mm to (132.1, 47.4)
- moved Q6 3.36 mm to (97.2, 58.4)
- moved Q4 2.86 mm to (120.6, 58.4)
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Routing:
- net +12V: track 0.00 -> 265.5 mm
- net GND: track 0.00 -> 154.7 mm
- net Net-(D5-A): track 0.00 -> 30.7 mm, vias 0 -> 2
- net Net-(D4-A): track 0.00 -> 28.8 mm, vias 0 -> 2
- net Net-(D3-A): track 0.00 -> 28.2 mm, vias 0 -> 2
- net Net-(D2-A): track 0.00 -> 27.7 mm, vias 0 -> 2
- net Net-(D1-A): track 0.00 -> 27.5 mm, vias 0 -> 2
- net Net-(D9-A): track 0.00 -> 21.1 mm
- net Net-(D8-A): track 0.00 -> 19.1 mm
- net Net-(D7-A): track 0.00 -> 16.0 mm
- net Net-(D6-A): track 0.00 -> 13.4 mm
- added copper zone on In2.Cu, net +5V
- added copper zone on In1.Cu, net GND
Other:
- board text added: "+5V"
- board text added: "GND"
