File: master_schematic/_autosave-master_schematic.kicad_sch (KiCad schematic)
At the start: 10 parts, among them J1 Conn_01x02_Shielded, SW1 SW_SPST, U1 RFM95, U2 teensy_4.1, U3 EA50 Power Converter

Commit message: added decoupling capacitors, fixed voltage values for TTs and load cells to +3V3
Parts:
- added J21: Conn_01x02_Shielded, hb_footprint_lib:AMASS_XT60PW-M, symbol Connector_Generic:Conn_01x02
Connections:
- net +5V: now also J21.1 (Pin_1)
- net GND: now also J21.2 (Pin_2)
