File: master_schematic/_autosave-master_schematic.kicad_pcb (KiCad board)
At the start: 4 copper layers, 157.5 x 111.9 mm, 84 parts, among them J1 12V Female, J10 0430450400, J11 1723103102, J12 1723103102, J13 1723103102, J14 1723103102, J15 1723103102, J16 1723103102, J17 1723103102, J18 1723103102, J19 1723103102, J2 0430450400, J20 1723103102, J21 5V Female, J3 0430450400, J4 0430450400, J5 0430450400, J6 0430450400, J7 0430450400, J8 0430450400, J9 0430450400, Q1 CWDM3011N TR13 PBFREE, Q10 CWDM3011N TR13 PBFREE, Q2 CWDM3011N TR13 PBFREE, Q3 CWDM3011N TR13 PBFREE, Q4 CWDM3011N TR13 PBFREE, Q5 CWDM3011N TR13 PBFREE, Q6 CWDM3011N TR13 PBFREE, Q7 CWDM3011N TR13 PBFREE, Q8 CWDM3011N TR13 PBFREE, Q9 CWDM3011N TR13 PBFREE, SW1 SW_SPST, U1 RFM95, U10 HX711, U11 HX711, U2 teensy_4.1, U4 MCP9600_Module, U5 MCP9600_Module, U6 MCP9600_Module, U7 MCP9600_Module, U8 MCP9600_Module, U9 HX711

Commit message: FINALLY FINISHED ThESE DAMN TRACES F&#%%%
Connections:
- U2 pad 5V: +5V -> (no net)
Routing:
- net /PV1_T: track 7.20 -> 100.3 mm, vias 1 -> 4
- net /SDA: track 76.5 -> 145.8 mm
- net /SCL: track 91.5 -> 134.6 mm
- net Net-(D8-A): track 0.00 -> 35.0 mm
- net +12V: track 0.00 -> 32.4 mm, vias 0 -> 10
- net Net-(D7-A): track 0.00 -> 31.9 mm
- net Net-(D6-A): track 0.00 -> 29.2 mm
- net /PT1_T: track 32.1 -> 60.4 mm, vias 0 -> 1
- net Net-(D5-A): track 0.01 -> 27.4 mm
- net Net-(D1-A): track 0.00 -> 25.2 mm
- net Net-(D4-A): track 0.00 -> 25.0 mm
- net Net-(D2-A): track 0.00 -> 24.2 mm
- net Net-(D3-A): track 0.00 -> 23.7 mm
- net Net-(D10-A): track 0.00 -> 21.7 mm
- net Net-(D9-A): track 0.00 -> 19.1 mm
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